File: _autosave-keebk75pcb.kicad_pcb (KiCad board)
At the start: 2 copper layers, 87.3 x 55.5 mm, 24 parts, among them SW1 SW_Push, U1 ATmega32U4-A, Y1 16MHz

Commit message: routing
Parts:
- F1, SW1, USB1: moved to B.Cu
- moved R1 15.7 mm to (65.1, 95.0)
- moved C3 9.61 mm to (74.6, 100.0)
- moved Y1 6.76 mm to (81.8, 100.0)
- moved R2 6.63 mm to (70.6, 95.0), turned to -90 degrees
- moved R3 6.51 mm to (60.3, 109.5), turned to 90 degrees
- moved C2 3.11 mm to (88.1, 100.0)
- turned F1 to -90 degrees
