File: keebk75pcb.kicad_sch (KiCad schematic)
At the start: 24 parts, among them SW1 SW_Push, U1 ATmega32U4-A, Y1 16MHz

Commit message: layout
Parts:
- renumbered MX3 to MX2, MX2 to MX3
Changed lines of the file:
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@@
   (symbol (lib_id "MX_Alps_Hybrid:MX-LED") (at 55.88 130.81 0) (unit 1)
     (in_bom yes) (on_board yes) (fields_autoplaced)
-    (property "Reference" "MX2" (id 0) (at 58.0356 124.46 0)
+    (property "Reference" "MX3" (id 0) (at 58.0356 124.46 0)
       (effects (font (size 1.524 1.524)))
     )
@@
   (symbol (lib_id "MX_Alps_Hybrid:MX-LED") (at 71.12 109.22 0) (unit 1)
     (in_bom yes) (on_board yes) (fields_autoplaced)
-    (property "Reference" "MX3" (id 0) (at 73.2756 102.87 0)
+    (property "Reference" "MX2" (id 0) (at 73.2756 102.87 0)
       (effects (font (size 1.524 1.524)))
     )
@@
       (reference "MX1") (unit 1) (value "MX-LED") (footprint "MX_Only:MXOnly-1U-Hotswap-LED")
     )
+    (path "/5ee9ead0-498c-4691-8e11-ec4be578bc9b"
+      (reference "MX2") (unit 1) (value "MX-LED") (footprint "MX_Only:MXOnly-1U-Hotswap-LED")
+    )
     (path "/24a25ee7-67e5-494b-a24f-d4cbee581e70"
-      (reference "MX2") (unit 1) (value "MX-LED") (footprint "MX_Only:MXOnly-1U-Hotswap-LED")
-    )
-    (path "/5ee9ead0-498c-4691-8e11-ec4be578bc9b"
       (reference "MX3") (unit 1) (value "MX-LED") (footprint "MX_Only:MXOnly-1U-Hotswap-LED")
     )

Commit message: gen
Other:
- moved on the sheet: C1, C4, C5, C6
Changed lines of the file:
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@@
   (junction (at 97.79 72.39) (diameter 0) (color 0 0 0 0)
   )
-  (junction (at 104.14 115.57) (diameter 0) (color 0 0 0 0)
-  )
   (junction (at 105.41 76.2) (diameter 0) (color 0 0 0 0)
   )
-  (junction (at 109.22 115.57) (diameter 0) (color 0 0 0 0)
-  )
-  (junction (at 109.22 110.49) (diameter 0) (color 0 0 0 0)
+  (junction (at 99.06 110.49) (diameter 0) (color 0 0 0 0)
   )
   (junction (at 106.68 110.49) (diameter 0) (color 0 0 0 0)
@@
   (junction (at 107.95 69.85) (diameter 0) (color 0 0 0 0)
   )
-  (junction (at 104.14 110.49) (diameter 0) (color 0 0 0 0)
-  )
   (junction (at 107.95 64.77) (diameter 0) (color 0 0 0 0)
   )
   (junction (at 49.53 143.51) (diameter 0) (color 0 0 0 0)
   )
+  (junction (at 99.06 115.57) (diameter 0) (color 0 0 0 0)
+  )
   (junction (at 134.62 143.51) (diameter 0) (color 0 0 0 0)
   )
@@
     (stroke (width 0) (type default) (color 0 0 0 0))
   )
+  (wire (pts (xy 106.68 115.57) (xy 115.57 115.57))
+    (stroke (width 0) (type default) (color 0 0 0 0))
+  )
   (wire (pts (xy 110.49 67.31) (xy 110.49 76.2))
     (stroke (width 0) (type default) (color 0 0 0 0))
@@
     (stroke (width 0) (type default) (color 0 0 0 0))
   )
-  (wire (pts (xy 104.14 110.49) (xy 106.68 110.49))
+  (wire (pts (xy 99.06 110.49) (xy 106.68 110.49))
     (stroke (width 0) (type default) (color 0 0 0 0))
   )
@@
     (stroke (width 0) (type default) (color 0 0 0 0))
   )
-  (wire (pts (xy 109.22 110.49) (xy 114.3 110.49))
-    (stroke (width 0) (type default) (color 0 0 0 0))
-  )
   (wire (pts (xy 54.61 134.62) (xy 49.53 135.89))
     (stroke (width 0) (type default) (color 0 0 0 0))
   )
-  (wire (pts (xy 106.68 115.57) (xy 109.22 115.57))
-    (stroke (width 0) (type default) (color 0 0 0 0))
-  )
   (wire (pts (xy 115.57 92.71) (xy 121.92 92.71))
     (stroke (width 0) (type default) (color 0 0 0 0))
   )
-  (wire (pts (xy 106.68 110.49) (xy 109.22 110.49))
-    (stroke (width 0) (type default) (color 0 0 0 0))
-  )
   (wire (pts (xy 102.87 62.23) (xy 107.95 62.23))
     (stroke (width 0) (type default) (color 0 0 0 0))
@@
     (stroke (width 0) (type default) (color 0 0 0 0))
   )
-  (wire (pts (xy 109.22 115.57) (xy 114.3 115.57))
-    (stroke (width 0) (type default) (color 0 0 0 0))
-  )
   (wire (pts (xy 134.62 52.07) (xy 137.16 52.07))
     (stroke (width 0) (type default) (color 0 0 0 0))
   )
+  (wire (pts (xy 106.68 110.49) (xy 115.57 110.49))
+    (stroke (width 0) (type default) (color 0 0 0 0))
+  )
   (wire (pts (xy 66.04 135.89) (xy 66.04 138.43))
     (stroke (width 0) (type default) (color 0 0 0 0))
@@
     (stroke (width 0) (type default) (color 0 0 0 0))
   )
-  (wire (pts (xy 99.06 110.49) (xy 104.14 110.49))
+  (wire (pts (xy 88.9 110.49) (xy 99.06 110.49))
     (stroke (width 0) (type default) (color 0 0 0 0))
   )
@@
     (stroke (width 0) (type default) (color 0 0 0 0))
   )
-  (wire (pts (xy 104.14 115.57) (xy 106.68 115.57))
-    (stroke (width 0) (type default) (color 0 0 0 0))
-  )
-  (wire (pts (xy 99.06 115.57) (xy 104.14 115.57))
+  (wire (pts (xy 99.06 115.57) (xy 106.68 115.57))
+    (stroke (width 0) (type default) (color 0 0 0 0))
+  )
+  (wire (pts (xy 88.9 115.57) (xy 99.06 115.57))
     (stroke (width 0) (type default) (color 0 0 0 0))
   )
@@
     (pin "2")
   )
-  (symbol (lib_id "Device:C_Small") (at 114.3 113.03 0) (unit 1)
-    (in_bom yes) (on_board yes) (fields_autoplaced)
-    (property "Reference" "C6" (id 0) (at 116.84 111.7662 0)
-      (effects (font (size 1.27 1.27)) (justify left))
-    )
-    (property "Value" "10uF" (id 1) (at 116.84 114.3062 0)
-      (effects (font (size 1.27 1.27)) (justify left))
-    )
-    (property "Footprint" "Capacitor_SMD:C_0805_2012Metric" (id 2) (at 114.3 113.03 0)
-      (effects (font (size 1.27 1.27)) hide)
-    )
-    (property "Datasheet" "~" (id 3) (at 114.3 113.03 0)
+  (symbol (lib_id "Device:C_Small") (at 115.57 113.03 0) (unit 1)
+    (in_bom yes) (on_board yes) (fields_autoplaced)
+    (property "Reference" "C6" (id 0) (at 118.11 111.7662 0)
+      (effects (font (size 1.27 1.27)) (justify left))
+    )
+    (property "Value" "10uF" (id 1) (at 118.11 114.3062 0)
+      (effects (font (size 1.27 1.27)) (justify left))
+    )
+    (property "Footprint" "Capacitor_SMD:C_0805_2012Metric" (id 2) (at 115.57 113.03 0)
+      (effects (font (size 1.27 1.27)) hide)
+    )
+    (property "Datasheet" "~" (id 3) (at 115.57 113.03 0)
       (effects (font (size 1.27 1.27)) hide)
     )
@@
     (pin "1")
   )
-  (symbol (lib_id "Device:C_Small") (at 109.22 113.03 0) (unit 1)
-    (in_bom yes) (on_board yes) (fields_autoplaced)
-    (property "Reference" "C5" (id 0) (at 111.76 111.7662 0)
-      (effects (font (size 1.27 1.27)) (justify left))
-    )
-    (property "Value" "0.1uF" (id 1) (at 111.76 114.3062 0)
-      (effects (font (size 1.27 1.27)) (justify left))
-    )
-    (property "Footprint" "Capacitor_SMD:C_0805_2012Metric" (id 2) (at 109.22 113.03 0)
-      (effects (font (size 1.27 1.27)) hide)
-    )
-    (property "Datasheet" "~" (id 3) (at 109.22 113.03 0)
+  (symbol (lib_id "Device:C_Small") (at 106.68 113.03 0) (unit 1)
+    (in_bom yes) (on_board yes) (fields_autoplaced)
+    (property "Reference" "C5" (id 0) (at 109.22 111.7662 0)
+      (effects (font (size 1.27 1.27)) (justify left))
+    )
+    (property "Value" "0.1uF" (id 1) (at 109.22 114.3062 0)
+      (effects (font (size 1.27 1.27)) (justify left))
+    )
+    (property "Footprint" "Capacitor_SMD:C_0805_2012Metric" (id 2) (at 106.68 113.03 0)
+      (effects (font (size 1.27 1.27)) hide)
+    )
+    (property "Datasheet" "~" (id 3) (at 106.68 113.03 0)
       (effects (font (size 1.27 1.27)) hide)
     )
@@
     (pin "1")
   )
-  (symbol (lib_id "Device:C_Small") (at 99.06 113.03 0) (unit 1)
+  (symbol (lib_id "Device:C_Small") (at 88.9 113.03 0) (unit 1)
     (in_bom yes) (on_board yes)
-    (property "Reference" "C1" (id 0) (at 101.6 111.7662 0)
-      (effects (font (size 1.27 1.27)) (justify left))
-    )
-    (property "Value" "0.1uF" (id 1) (at 101.6 114.3062 0)
-      (effects (font (size 1.27 1.27)) (justify left))
-    )
-    (property "Footprint" "Capacitor_SMD:C_0805_2012Metric" (id 2) (at 99.06 113.03 0)
-      (effects (font (size 1.27 1.27)) hide)
-    )
-    (property "Datasheet" "~" (id 3) (at 99.06 113.03 0)
+    (property "Reference" "C1" (id 0) (at 91.44 111.7662 0)
+      (effects (font (size 1.27 1.27)) (justify left))
+    )
+    (property "Value" "0.1uF" (id 1) (at 91.44 114.3062 0)
+      (effects (font (size 1.27 1.27)) (justify left))
+    )
+    (property "Footprint" "Capacitor_SMD:C_0805_2012Metric" (id 2) (at 88.9 113.03 0)
+      (effects (font (size 1.27 1.27)) hide)
+    )
+    (property "Datasheet" "~" (id 3) (at 88.9 113.03 0)
       (effects (font (size 1.27 1.27)) hide)
     )
@@
     (pin "2")
   )
-  (symbol (lib_id "Device:C_Small") (at 104.14 113.03 0) (unit 1)
-    (in_bom yes) (on_board yes) (fields_autoplaced)
-    (property "Reference" "C4" (id 0) (at 106.68 111.7662 0)
-      (effects (font (size 1.27 1.27)) (justify left))
-    )
-    (property "Value" "0.1uF" (id 1) (at 106.68 114.3062 0)
-      (effects (font (size 1.27 1.27)) (justify left))
-    )
-    (property "Footprint" "Capacitor_SMD:C_0805_2012Metric" (id 2) (at 104.14 113.03 0)
-      (effects (font (size 1.27 1.27)) hide)
-    )
-    (property "Datasheet" "~" (id 3) (at 104.14 113.03 0)
-      (effects (font (size 1.27 1.27)) hide)
-    )
+  (symbol (lib_id "Device:C_Small") (at 99.06 113.03 0) (unit 1)
+    (in_bom yes) (on_board yes) (fields_autoplaced)
+    (property "Reference" "C4" (id 0) (at 101.6 111.7662 0)
+      (effects (font (size 1.27 1.27)) (justify left))
+    )
+    (property "Value" "0.1uF" (id 1) (at 101.6 114.3062 0)
+      (effects (font (size 1.27 1.27)) (justify left))
+    )
+    (property "Footprint" "Capacitor_SMD:C_0805_2012Metric" (id 2) (at 99.06 113.03 0)
+      (effects (font (size 1.27 1.27)) hide)
+    )
+    (property "Datasheet" "~" (id 3) (at 99.06 113.03 0)
+      (effects (font (size 1.27 1.27)) hide)
+    )
