File: keebk75pcb.kicad_pcb (KiCad board)
At the start: 2 copper layers, 85.8 x 50 mm, 24 parts, among them SW1 SW_Push, U1 ATmega32U4-A, Y1 16MHz

Commit message: fin
Connections:
- U1 pad 27: unconnected-(U1-Pad27) -> Row0
- U1 pad 28: unconnected-(U1-Pad28) -> Col1
- U1 pad 29: unconnected-(U1-Pad29) -> Col0
- U1 pad 30: unconnected-(U1-Pad30) -> Row1
Routing:
- net Row0: track 0.00 -> 55.7 mm, vias 0 -> 4
- net Col1: track 19.1 -> 49.3 mm, vias 0 -> 2
- net Row1: track 19.9 -> 48.3 mm
- net Col0: track 19.0 -> 30.7 mm
